Commit message: Forearm is OK.

File: urdf/px150_coll.urdf (robot description, URDF)
Before this commit: robot px150, 13 links, 12 joints
Joints:
- joint elbow: origin xyz=0.05 0 0.15 rpy=0 0 0 -> xyz=0.05 0 -0.15 rpy=0 3.141592653589793 0

Commit message: Wrist OK. Why a shoulder rotation of 1 gives 90 degrees?

File: urdf/px150_coll.urdf (robot description, URDF)
Before this commit: robot px150, 13 links, 12 joints
Joints:
- joint wrist_angle: origin xyz=0.15 0 0 rpy=0 0 0 -> xyz=0.15 0 0 rpy=0 0 3.141592653589793

Commit message: Bugfix for rotational joints.

File: urdf/px150_coll.urdf (robot description, URDF)
Before this commit: robot px150, 13 links, 12 joints
Joints:
- joint elbow: origin xyz=0.05 0 -0.15 rpy=0 3.141592653589793 0 -> xyz=0.05 0 0.15 rpy=0 0 0
- joint wrist_angle: origin xyz=0.15 0 0 rpy=0 0 3.141592653589793 -> xyz=0.15 0 0 rpy=0 0 0

Commit message: Made the URDF Gazebo-compatible.

File: urdf/px150_coll.urdf (robot description, URDF)
Before this commit: robot px150, 13 links, 12 joints
Links:
- added link world
Joints:
- added joint fix_to_world: type fixed, parent world, child px150/base_link
